Commit message: update structures

File: examples/assets/robots/franka_panda/panda_arm.urdf (robot description, URDF)
Before this commit: robot panda, 22 links, 21 joints
Links:
- removed link panda_hand_sc
- removed link panda_hand_tcp
- removed link panda_leftfinger
- removed link panda_rightfinger
Joints:
- removed joint panda_finger_joint1
- removed joint panda_finger_joint2
- removed joint panda_hand_sc_joint
- removed joint panda_hand_tcp_joint
